File: pcb/Macropad_Kicad_Project/macropad_v01.kicad_pcb (KiCad board)
At the start: 2 copper layers, 65 parts, among them J2 Expansion-Connector, K1 KEYSW, K10 KEYSW, K11 KEYSW, K12 KEYSW, K13 KEYSW, K14 KEYSW, K15 KEYSW, K16 KEYSW-canadian_parts-yampad_v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, K17 KEYSW-canadian_parts-yampad_v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

Commit message: PCB DONE!!!
(i think)
Parts:
- added C11: macropad_v01-rescue_Symbols-Cache_Device_C-Symbols-Cache, Footprints:Capacitor-(100uF), F.Cu at (97.8, 133.3)
- added C12: Device_C-Symbols-Cache, Footprints:Capacitor-(100uF), F.Cu at (95.2, 108.0)
- moved C8 140.9 mm to (120.7, 127.6), turned to 270 degrees
- moved C9 127.4 mm to (120.7, 108.6), turned to 270 degrees
- moved C1 122.3 mm to (120.7, 70.5), turned to 270 degrees
- moved C7 112.2 mm to (139.7, 127.6), turned to 270 degrees
- moved C3 102.3 mm to (158.8, 70.5), turned to 270 degrees
- moved C4 85.0 mm to (158.8, 89.5), turned to 270 degrees
- moved C10 69.2 mm to (120.7, 89.5), turned to 270 degrees
- moved C2 60.2 mm to (139.7, 70.5), turned to 270 degrees
- moved J2 16.5 mm to (94.0, 120.7)
- moved U2 5.72 mm to (95.2, 139.1)
Connections:
- K16 pad 1: Net-(K16-Pad1) -> COL3
- K17 pad 1: Net-(K16-Pad1) -> COL3
- K18 pad 1: Net-(K16-Pad1) -> COL3
- K19 pad 1: Net-(K16-Pad1) -> COL3
- K20 pad 1: Net-(K16-Pad1) -> COL3
Routing:
- net VCC: track 7.62 -> 316.4 mm, vias 0 -> 8
- net COL3: track 0.00 -> 192.1 mm, vias 0 -> 6
- net COL2: track 0.00 -> 168.6 mm, vias 0 -> 6
- net COL1: track 0.00 -> 147.7 mm, vias 0 -> 6
- net ROW4: track 0.00 -> 126.8 mm, vias 0 -> 2
- net COL0: track 0.00 -> 125.7 mm, vias 0 -> 6
- net GND: track 20.5 -> 145.8 mm, vias 0 -> 4
- net ROW3: track 0.00 -> 111.6 mm, vias 0 -> 2
- net ROW2: track 0.00 -> 94.1 mm, vias 0 -> 2
- net IR: track 0.00 -> 77.8 mm
- net ROW0: track 0.00 -> 77.4 mm
- net ROW1: track 0.00 -> 77.3 mm
- net TX: track 0.00 -> 74.1 mm, vias 0 -> 2
- net RX: track 0.90 -> 71.4 mm, vias 0 -> 2
- net A2: track 0.00 -> 65.2 mm
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- added copper zone on B.Cu, net GND
- added copper zone on F.Cu, net GND
Other:
- board outline added: 95.9 x 96.5 mm
- board text added: "Created by Ahmed Hafeez-Baig (github.com/Baigel/Macropad) Forked from github.com/mattdibi/yampad"
- board text added: "IR Sensor"
