File: pcb/Macropad_Kicad_Project/macropad_v01.sch (KiCad schematic (older format))
At the start: 65 parts, among them J2 Expansion-Connector, K1 KEYSW, K10 KEYSW, K11 KEYSW, K12 KEYSW, K13 KEYSW, K14 KEYSW, K15 KEYSW, K16 KEYSW-canadian_parts-yampad_v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, K17 KEYSW-canadian_parts-yampad_v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

Commit message: PCB DONE!!!
(i think)
Parts:
- added C11: macropad_v01-rescue_Symbols-Cache_Device_C-Symbol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, Footprints:Capacitor-(100uF), symbol Symbols-Cache:macropad_v01-rescue_Symbols-Cache_Device_C-Symbols-Cache
- added C12: Device_C-Symbols-Cache, Footprints:Capacitor-(100uF), symbol macropad_v01-rescue:Device_C-Symbols-Cache
- C10, C9: symbol Symbols-Cache:Symbols-Cache_Device_C -> macropad_v01-rescue:Symbols-Cache_Device_C-Symbols-Cache
Connections:
- net COL3: now also K16.1, K17.1, K18.1, K19.1, K20.1
- net GND: now also C11.1, C12.1
- net VCC: now also C11.2, C12.2
Other:
- moved on the sheet: U2
